File: Kicad/Qubit Control Board.kicad_sch (KiCad schematic)
At the start: 128 parts, among them J1 USB_C_Receptacle_PowerOnly_6P, J2 CLK_Pins, J3 Idata, J4 Qdata, J5 SPIdata, J6 SMA, U2 TRF372017IRGZR, U3 LT1963AxST-3.3, U4 LT1963AxST-1.8, U5 SN65LVDS1DBV, U6 AD9743BCPZ, Y1 SiT8008xx-3x-xxN

Commit message: added footprints
Parts:
- added RDIFF2, RDIFF3: 100R, symbol Device:R
- U2: footprint RGZ48_5P6X5P6 -> footprints789:RGZ48_5P6X5P6
- U6: footprint CP-72-1_ADI -> footprints789:CP-72-1_ADI-M
Connections:
- net at CCQN.2, U2.9 (BBQ_N): now also RDIFF2.2
- net at CCIP1.2, U2.27 (BBI_P): now also RDIFF3.1
- net at CCQP.2, U2.10 (BBQ_P): now also RDIFF2.1
- net at CCIN1.2, U2.28 (BBI_N): now also RDIFF3.2

Commit message: added CRC filter after the DAC
Parts:
- removed CINF, CIPF, CQNF, CQPF: 100p, symbol Device:C
- added CIF1, CIF2, CQF1, CQF2: 130p, symbol Device:C
- RINF, RIPF, RQNF, RQPF: value 49.9R -> 33R
Connections:
- net BBIN: now also CIF2.2
- net BBIP: now also CIF2.1
- net BBQN: now also CQF2.2
- net BBQP: now also CQF2.1
- net IOUTN: now also CIF1.2
- net IOUTP: now also CIF1.1
- net QOUTN: now also CQF1.2
- net QOUTP: now also CQF1.1
Other:
- moved on the sheet: RINF, RIPF, RLOAD1, RLOAD2, RLOAD3, RLOAD4, RQNF, RQPF

Commit message: put in most footprints
Parts:
- CBULK1, CBULK3, CBULK5, CBULK7, CIN1, CLDO1, CLDO2, CLDO3, CLDO4: footprint (none) -> Capacitor_SMD:C_1206_3216Metric_Pad1.33x1.80mm_HandSolder
- CBULK2, CBULK4, CBULK6, CBULK8, CD11, CD20, CD21, CD22, CD26: footprint (none) -> Capacitor_SMD:C_0805_2012Metric_Pad1.18x1.45mm_HandSolder
- CC1, CC2, CCDAC1, CCDAC2, CCIN1, CCIP1, CD1, CD10, CD12, CD13, CD14, CD15, CD16, CD17, CD18, CD19, CD2, CD23, CD24, CD25, CD27, CD28, CD29, CD3, CD4, CD5, CD6, CD7, CD8, CD9, CDC1, CIF1, CIF2, CIN2, CLF1, CLF2, CLF3, CQF1, CQF2, CRE1: footprint (none) -> Capacitor_SMD:C_0603_1608Metric
- CCQN1: renamed from CCQN; footprint (none) -> Capacitor_SMD:C_0603_1608Metric
- CCQP1: renamed from CCQP; footprint (none) -> Capacitor_SMD:C_0603_1608Metric
- FB1, FB2, FB3, FB4: footprint (none) -> Inductor_SMD:L_0603_1608Metric_Pad1.05x0.95mm_HandSolder
- J2: footprint (none) -> Connector_PinHeader_1.00mm:PinHeader_1x02_P1.00mm_Vertical
- J3, J4: footprint (none) -> Connector_PinHeader_1.00mm:PinHeader_1x11_P1.00mm_Vertical
- J5: footprint (none) -> Connector_PinHeader_1.00mm:PinHeader_1x06_P1.00mm_Vertical
- J6: footprint (none) -> Connector_Coaxial:SMA_Molex_73251-1153_EdgeMount_Horizontal
- RAP1, RAP2, RAP3, RDIFF1, RDIFF2, RDIFF3, RDIFF4, RDIV1, RDIV2, RFS1, RLF1, RLF2, RLOAD1, RLOAD2, RLOAD3, RLOAD4, RPD1, RPD2, RPD3, RS1, Rd1, Rd2: footprint (none) -> Resistor_SMD:R_0603_1608Metric
- RID0, RID1, RID2, RID3, RID4, RID5, RID6, RID7, RID8, RID9, RQD0, RQD1, RQD2, RQD3, RQD4, RQD5, RQD6, RQD7, RQD8, RQD9, RT1, RT2, RTSPI1, RTSPI2, RTSPI3, RTSPI4, RTSPI5: footprint (none) -> Resistor_SMD:R_0603_1608Metric_Pad0.98x0.95mm_HandSolder
- RINF1: renamed from RINF; footprint (none) -> Resistor_SMD:R_0603_1608Metric_Pad0.98x0.95mm_HandSolder
- RIPF1: renamed from RIPF; footprint (none) -> Resistor_SMD:R_0603_1608Metric_Pad0.98x0.95mm_HandSolder
- RQNF1: renamed from RQNF; footprint (none) -> Resistor_SMD:R_0603_1608Metric_Pad0.98x0.95mm_HandSolder
- RQPF1: renamed from RQPF; footprint (none) -> Resistor_SMD:R_0603_1608Metric_Pad0.98x0.95mm_HandSolder

Commit message: changed oss and updated footprint sizes on de caps
Parts:
- removed Y1: SiT8008xx-3x-xxN, Oscillator:Oscillator_SMD_SiT_PQFN-4Pin_5.0x3.2mm, symbol Oscillator:SiT8008xx-3x-xxN
- added Y2: CVHD-950-100.000, footprints789:OSCSC508P1420X914X530-4N, symbol CVHD-950-100.000:CVHD-950-100.000
- CD1, CD10, CD12, CD13, CD14, CD15, CD16, CD17, CD18, CD19, CD2, CD23, CD24, CD25, CD27, CD29, CD3, CD4, CD5, CD6, CD7, CD8, CD9, CDC1, CIN2: footprint Capacitor_SMD:C_0603_1608Metric -> Capacitor_SMD:C_0402_1005Metric
- J1: footprint (none) -> Connector_USB:USB_C_Receptacle_GCT_USB4135-GF-A_6P_TopMnt_Horizontal
- RID0, RID1, RID2, RID3, RID4, RID5, RID6, RID7, RID8, RID9, RQD0, RQD1, RQD2, RQD3, RQD4, RQD5, RQD6, RQD7, RQD8, RQD9, RT1, RT2, RTSPI1, RTSPI2, RTSPI3, RTSPI4, RTSPI5: footprint Resistor_SMD:R_0603_1608Metric_Pad0.98x0.95mm_HandSolder -> Resistor_SMD:R_0402_1005Metric
- RINF1, RIPF1, RQNF1, RQPF1: footprint Resistor_SMD:R_0603_1608Metric_Pad0.98x0.95mm_HandSolder -> Resistor_SMD:R_0603_1608Metric
Connections:
- net +3.3V: now also Y2.1 (CTRL), Y2.4 (VDD)
- net GND: now also Y2.2 (GND)
- net at RT2.1: now also Y2.3 (OUT)
Other:
- note removed: "F_c = 31.895 MHz"
- moved on the sheet: CC1, RT2

Commit message: diff clock routing
Parts:
- CD2, CD3: footprint Capacitor_SMD:C_0402_1005Metric -> Capacitor_SMD:C_0201_0603Metric
- CD28: footprint Capacitor_SMD:C_0603_1608Metric -> Capacitor_SMD:C_0402_1005Metric
Changed lines of the file:
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@@
 			)
 		)
-		(property "Footprint" "Capacitor_SMD:C_0402_1005Metric"
+		(property "Footprint" "Capacitor_SMD:C_0201_0603Metric"
 			(at 153.9748 176.53 0)
 			(hide yes)
@@
 			)
 		)
-		(property "Footprint" "Capacitor_SMD:C_0402_1005Metric"
+		(property "Footprint" "Capacitor_SMD:C_0201_0603Metric"
 			(at 165.4048 176.53 0)
 			(hide yes)
@@
 			)
 		)
-		(property "Footprint" "Capacitor_SMD:C_0603_1608Metric"
+		(property "Footprint" "Capacitor_SMD:C_0402_1005Metric"
 			(at 161.5948 331.47 0)
 			(hide yes)

Commit message: Finished diff clock routing
Parts:
- F1: footprint (none) -> Fuse:Fuse_1206_3216Metric
Changed lines of the file:
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@@
 			)
 		)
-		(property "Footprint" ""
+		(property "Footprint" "Fuse:Fuse_1206_3216Metric"
 			(at 78.74 65.278 90)
 			(hide yes)

Commit message: routed USBC
Parts:
- removed RS1: 0R, Resistor_SMD:R_0603_1608Metric, symbol Device:R
Connections:
- net GND: now also J1.SH (SHIELD)
Changed lines of the file:
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@@
 	)
 	(junction
+		(at 54.61 99.06)
+		(diameter 0)
+		(color 0 0 0 0)
+	)
+	(junction
 		(at 509.27 185.42)
 		(diameter 0)
@@
 	)
 	(junction
-		(at 54.61 99.06)
-		(diameter 0)
-		(color 0 0 0 0)
-	)
-	(junction
 		(at 398.78 231.14)
 		(diameter 0)
@@
 	(wire
 		(pts
-			(xy 54.61 99.06) (xy 54.61 106.68)
-		)
-		(stroke
-			(width 0)
-			(type default)
-		)
-	)
-	(wire
-		(pts
 			(xy 406.4 172.72) (xy 417.83 172.72)
 		)
@@
 	(wire
 		(pts
+			(xy 46.99 99.06) (xy 54.61 99.06)
+		)
+		(stroke
+			(width 0)
+			(type default)
+		)
+	)
+	(wire
+		(pts
 			(xy 175.26 328.93) (xy 193.04 328.93)
 		)
@@
 	(wire
 		(pts
+			(xy 54.61 99.06) (xy 54.61 106.68)
+		)
+		(stroke
+			(width 0)
+			(type default)
+		)
+	)
+	(wire
+		(pts
 			(xy 85.09 170.18) (xy 85.09 172.72)
 		)
@@
 					(unit 1)
 				)
-			)
-		)
-	)
-	(symbol
-		(lib_id "Device:R")
-		(at 50.8 99.06 90)
-		(unit 1)
-		(body_style 1)
-		(exclude_from_sim no)
-		(in_bom yes)
-		(on_board yes)
-		(in_pos_files yes)
-		(dnp no)
-		(property "Reference" "RS1"
-			(at 50.8 93.726 90)
-			(show_name no)
-			(do_not_autoplace no)
-			(effects
-				(font
-					(size 1.27 1.27)
-				)
-			)
-		)
-		(property "Value" "0R"
-			(at 50.8 96.266 90)
-			(show_name no)
-			(do_not_autoplace no)
-			(effects
-				(font
-					(size 1.27 1.27)
-				)
-			)
-		)
-		(property "Footprint" "Resistor_SMD:R_0603_1608Metric"
-			(at 50.8 100.838 90)
-			(hide yes)
-			(show_name no)
-			(do_not_autoplace no)
-			(effects
-				(font
-					(size 1.27 1.27)
-				)
-			)
-		)
-		(property "Datasheet" ""
-			(at 50.8 99.06 0)
-			(hide yes)
-			(show_name no)
-			(do_not_autoplace no)
-			(effects
-				(font
-					(size 1.27 1.27)
-				)
-			)
-		)
-		(property "Description" "Resistor"
-			(at 50.8 99.06 0)
-			(hide yes)
-			(show_name no)
-			(do_not_autoplace no)
-			(effects
-				(font
-					(size 1.27 1.27)
-				)
-			)
-		)
-		(pin "1"
-		)
-		(pin "2"
-		)
-		(instances
-			(project "Qubit Control Board"
-				(path "/d02a9e30-46b8-444a-9e12-1a93fb154b6d"
-					(reference "RS1")
-					(unit 1)
-				)

Commit message: updated LDO power set up
Parts:
- removed U3: LT1963AxST-3.3, Package_TO_SOT_SMD:SOT-223-3_TabPin2, symbol Regulator_Linear:LT1963AxST-3.3
- removed U4: LT1963AxST-1.8, Package_TO_SOT_SMD:SOT-223-3_TabPin2, symbol Regulator_Linear:LT1963AxST-1.8
- added CD30, CD31, CD32, CD33, CD34, CD35, CSEN1, CSEN2, CSEN3: 100n, Capacitor_SMD:C_0402_1005Metric, symbol Device:C
- added CLDO5: 10u, Capacitor_SMD:C_1206_3216Metric_Pad1.33x1.80mm_HandSolder, symbol Device:C
- added CLDOS1, CLDOS2, CLDOS3: 470n, Capacitor_SMD:C_0402_1005Metric, symbol Device:C
- added RLDOS1, RLDOS2: 33.2k, Resistor_SMD:R_0603_1608Metric, symbol Device:R
- added RLDOS3: 17.8k, Resistor_SMD:R_0603_1608Metric, symbol Device:R
- added U1, U3, U4: LT3045xMSE, Package_SO:MSOP-12-1EP_3x4.039mm_P0.65mm_EP1.651x2.845mm, symbol Regulator_Linear:LT3045xMSE
Connections:
- net +1.8V: now also CD35.2, CSEN3.2, U4.10 (OUTS), U4.11 (OUT), U4.12 (OUT); no longer CLDO4.1
- net +5V: now also CLDO2.1, CLDO4.1, CD30.2, CD32.2, CD34.2, CLDO5.1, U1.1 (IN), U1.2 (IN), U1.3 (IN), U1.4 (EN/UV), U1.7 (PGFB), U3.1 (IN), U3.2 (IN), U3.3 (IN), U3.4 (EN/UV), U3.7 (PGFB), U4.1 (IN), U4.2 (IN), U4.3 (IN), U4.4 (EN/UV), U4.7 (PGFB)
- net GND: now also CD30.1, CD31.1, CD32.1, CD33.1, CD34.1, CD35.1, CLDO5.2, CLDOS1.1, CLDOS2.1, CLDOS3.1, CSEN1.1, CSEN2.1, CSEN3.1, RLDOS1.1, RLDOS2.1, RLDOS3.1, U1.13 (GND), U1.6 (ILIM), U1.9 (GND), U3.13 (GND), U3.6 (ILIM), U3.9 (GND), U4.13 (GND), U4.6 (ILIM), U4.9 (GND)
- net +3.3V renamed +3.3V-A
- net +3.3V-A: now also CD31.2, CSEN1.2, U1.10 (OUTS), U1.11 (OUT), U1.12 (OUT); no longer CBULK7.1, CBULK8.1, CD10.2, CD11.2, CLDO2.1, FB2.1, FB3.1, FB4.1, Y2.1 (CTRL), Y2.4 (VDD)
- new net: CLDOS3.2, RLDOS3.2, U4.8 (SET)
- new net: CLDOS2.2, RLDOS2.2, U3.8 (SET)
- new net: CLDOS1.2, RLDOS1.2, U1.8 (SET)
- new net +3.3V-B: CBULK7.1, CBULK8.1, CD10.2, CD11.2, CD33.2, CSEN2.2, FB2.1, FB3.1, FB4.1, U3.10 (OUTS), U3.11 (OUT), U3.12 (OUT), Y2.1 (CTRL), Y2.4 (VDD)
- no-connect marks 26 -> 29
Other:
- moved on the sheet: CBULK1, CBULK2, CBULK3, CBULK4, CC2, CCDAC1, CCDAC2, CD1, CD2, CD28, CD29, CD3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
